Commit message: modify

File: urdf/models/kinect.urdf (robot description, URDF)
Before this commit: robot camera, 3 links, 2 joints
Joints:
- joint joint_kinect: origin xyz=0 0 0 rpy=0 0 0 -> xyz=1.0 0.0 0.5 rpy=0.0 0.35 3.14

Commit message: add files to make datasets automatically

File: urdf/models/kinect.urdf (robot description, URDF)
Before this commit: robot camera, 3 links, 2 joints
Joints:
- joint joint_kinect: origin xyz=1.0 0.0 0.5 rpy=0.0 0.35 3.14 -> xyz=1.0 0.0 0.5 rpy=0.0 0.35 -3.14
