Commit message: [add] make auto datasets generator with occulusion

File: urdf/models/obstacle_box.urdf (robot description, URDF)
Before this commit: robot camera, 2 links, 1 joints
Links:
- link object_link: geometry visual box size=0.22 0.22 0.22

File: urdf/models/obstacle_box_small.urdf (robot description, URDF)
Before this commit: robot camera, 2 links, 1 joints
Links:
- link object_link: geometry visual box size=0.07 0.07 0.07
