Commit message: modify collision and origin

File: urdf/models/hv8.urdf (robot description, URDF)
Before this commit: robot camera, 2 links, 1 joints
Links:
- link object_link: geometry collision mesh filename=package://kinect_bringup/meshes/HV8.STL; visual mesh filename=package://kinect_bringup/meshes/HV8.STL

File: urdf/models/kinect.urdf (robot description, URDF)
Before this commit: robot camera, 3 links, 2 joints
Joints:
- joint joint_kinect: origin xyz=1.0 0.0 0.5 rpy=0.0 0.35 -3.14 -> xyz=0.0 0.0 0.0 rpy=0.0 0.0 0.0
