Commit message: Fix project name from kinect_bringup to datasets_generator

File: urdf/models/hv6.urdf (robot description, URDF)
Before this commit: robot camera, 2 links, 1 joints
Links:
- link object_link: geometry collision box size=0.065 0.25 0.082; visual mesh filename=package://datasets_generator/meshes/HV6.stl

File: urdf/models/hv7.urdf (robot description, URDF)
Before this commit: robot camera, 2 links, 1 joints
Links:
- link object_link: geometry collision box size=0.025 0.25 0.022; visual mesh filename=package://datasets_generator/meshes/HV7.stl

File: urdf/models/hv8.urdf (robot description, URDF)
Before this commit: robot camera, 2 links, 1 joints
Links:
- link object_link: geometry collision mesh filename=package://datasets_generator/meshes/HV8.STL; visual mesh filename=package://datasets_generator/meshes/HV8.STL

File: urdf/models/object.urdf (robot description, URDF)
Before this commit: robot camera, 2 links, 1 joints
Links:
- link object_link: geometry collision box size=0.065 0.25 0.082; visual mesh filename=package://datasets_generator/meshes/object.stl

File: urdf/models/object.urdf.xacro (robot description, xacro)
@@ -5,5 +5,5 @@
       <visual>
         <geometry>
-          <mesh filename="package://kinect_bringup/meshes/HV6.stl"/>
+          <mesh filename="package://datasets_generator/meshes/HV6.stl"/>
         </geometry>
         <material name="red"/>
